File: first_design/first_design.sch (KiCad schematic (older format))
At the start: 52 parts, among them J1 Conn_02x20_Odd_Even, J2 Accelerometer_small, J3 Accelerometer_standard, J4 Servo_motor, SW1 SW_DPST, SW2 SW_DPST, SW3 SW_DPST, SW4 SW_DPST

Commit message: footprints added
Parts:
- 2N7002K1, 2N7002K2: footprint Package_TO_SOT_SMD:SOT-23 -> library_express_pro:SOT23
- AI-1223-TWT-5V-5-R1: footprint (none) -> library_express_pro:Buzzer_AI-1223-TWT-5V-5-R
- MotorController1: footprint Package_SO:SOIC-16_3.9x9.9mm_P1.27mm -> library_express_pro:SO-16N
- R1, R10, R11, R12, R13, R14, R1_buck1, R2, R2_buck1, R3, R4, R5, R7, R8, R9, R_IR1, Rmax1: footprint (none) -> library_express_pro:R_1.2mm
- Si4101DY1: renamed from SPD30P06P_G1; footprint Package_TO_SOT_SMD:TO-252-2 -> library_express_pro:SOT23
- StepDownConverter1: footprint Package_SO:Diodes_SO-8EP -> library_express_pro:SO-8
- VoltageMonitor1: footprint (none) -> library_express_pro:SSOP3
Changed lines of the file:
@@
 F 0 "Rmax1" H 720 1196 50  0000 L CNN
 F 1 "280" H 720 1105 50  0000 L CNN
-F 2 "" V 580 1150 50  0001 C CNN
+F 2 "library_express_pro:R_1.2mm" V 580 1150 50  0001 C CNN
 F 3 "~" H 650 1150 50  0001 C CNN
 	1    650  1150
@@
 F 0 "MotorController1" H 9650 1875 50  0000 C CNN
 F 1 "VNH7070BAS" H 9650 1784 50  0000 C CNN
-F 2 "Package_SO:SOIC-16_3.9x9.9mm_P1.27mm" H 9650 850 50  0001 C CNN
+F 2 "library_express_pro:SO-16N" H 9650 850 50  0001 C CNN
 F 3 "" H 9650 850 50  0001 C CNN
 	1    9650 1250
@@
 F 0 "StepDownConverter1" H 4925 1865 50  0000 C CNN
 F 1 "AP65450" H 4925 1774 50  0000 C CNN
-F 2 "Package_SO:Diodes_SO-8EP" H 5350 1100 50  0001 C CNN
+F 2 "library_express_pro:SO-8" H 5350 1100 50  0001 C CNN
 F 3 "" H 5350 1100 50  0001 C CNN
 	1    4950 1350
@@
 F 0 "R3" V 4607 1400 50  0000 C CNN
 F 1 "100K" V 4516 1400 50  0000 C CNN
-F 2 "" V 4330 1400 50  0001 C CNN
+F 2 "library_express_pro:R_1.2mm" V 4330 1400 50  0001 C CNN
 F 3 "~" H 4400 1400 50  0001 C CNN
 	1    4400 1400
@@
 F 0 "R2_buck1" V 6307 2150 50  0001 C CNN
 F 1 "22.1K" V 6216 2150 50  0000 C CNN
-F 2 "" V 6030 2150 50  0001 C CNN
+F 2 "library_express_pro:R_1.2mm" V 6030 2150 50  0001 C CNN
 F 3 "~" H 6100 2150 50  0001 C CNN
 	1    6100 2150
@@
 F 0 "R1_buck1" V 5893 1800 50  0001 C CNN
 F 1 "124k" V 5984 1800 50  0000 C CNN
-F 2 "" V 6030 1800 50  0001 C CNN
+F 2 "library_express_pro:R_1.2mm" V 6030 1800 50  0001 C CNN
 F 3 "~" H 6100 1800 50  0001 C CNN
 	1    6100 1800
@@
 F 0 "2N7002K2" H 2306 3196 50  0000 L CNN
 F 1 "NMOS_DGS" H 2306 3105 50  0000 L CNN
-F 2 "Package_TO_SOT_SMD:SOT-23" H 2300 3250 50  0001 C CNN
+F 2 "library_express_pro:SOT23" H 2300 3250 50  0001 C CNN
 F 3 "~" H 2100 3150 50  0001 C CNN
 	1    2100 3150
@@
 F 0 "R5" V 1693 3350 50  0001 C CNN
 F 1 "10K" H 1784 3350 50  0000 C CNN
-F 2 "" V 1830 3350 50  0001 C CNN
+F 2 "library_express_pro:R_1.2mm" V 1830 3350 50  0001 C CNN
 F 3 "~" H 1900 3350 50  0001 C CNN
 	1    1900 3350
@@
 F 0 "R8" H 4570 5896 50  0001 L CNN
 F 1 "220" H 4430 5850 50  0000 R CNN
-F 2 "" V 4430 5850 50  0001 C CNN
+F 2 "library_express_pro:R_1.2mm" V 4430 5850 50  0001 C CNN
 F 3 "~" H 4500 5850 50  0001 C CNN
 	1    4500 5850
@@
 F 0 "R7" H 4570 5096 50  0001 L CNN
 F 1 "220" H 4430 5050 50  0000 R CNN
-F 2 "" V 4430 5050 50  0001 C CNN
+F 2 "library_express_pro:R_1.2mm" V 4430 5050 50  0001 C CNN
 F 3 "~" H 4500 5050 50  0001 C CNN
 	1    4500 5050
@@
 F 0 "R9" H 4570 6646 50  0001 L CNN
 F 1 "220" H 4430 6600 50  0000 R CNN
-F 2 "" V 4430 6600 50  0001 C CNN
+F 2 "library_express_pro:R_1.2mm" V 4430 6600 50  0001 C CNN
 F 3 "~" H 4500 6600 50  0001 C CNN
 	1    4500 6600
@@
 F 0 "R10" H 4570 7446 50  0001 L CNN
 F 1 "220" H 4430 7400 50  0000 R CNN
-F 2 "" V 4430 7400 50  0001 C CNN
+F 2 "library_express_pro:R_1.2mm" V 4430 7400 50  0001 C CNN
 F 3 "~" H 4500 7400 50  0001 C CNN
 	1    4500 7400
@@
 F 0 "R11" H 6370 5746 50  0001 L CNN
 F 1 "82" H 6230 5700 50  0000 R CNN
-F 2 "" V 6230 5700 50  0001 C CNN
+F 2 "library_express_pro:R_1.2mm" V 6230 5700 50  0001 C CNN
 F 3 "~" H 6300 5700 50  0001 C CNN
 	1    6300 5700
@@
 F 0 "R12" H 6370 6296 50  0001 L CNN
 F 1 "82" H 6230 6250 50  0000 R CNN
-F 2 "" V 6230 6250 50  0001 C CNN
+F 2 "library_express_pro:R_1.2mm" V 6230 6250 50  0001 C CNN
 F 3 "~" H 6300 6250 50  0001 C CNN
 	1    6300 6250
@@
 F 0 "R13" H 6370 6846 50  0001 L CNN
 F 1 "82" H 6230 6800 50  0000 R CNN
-F 2 "" V 6230 6800 50  0001 C CNN
+F 2 "library_express_pro:R_1.2mm" V 6230 6800 50  0001 C CNN
 F 3 "~" H 6300 6800 50  0001 C CNN
 	1    6300 6800
@@
 F 0 "R14" H 6370 7346 50  0001 L CNN
 F 1 "82" H 6230 7300 50  0000 R CNN
-F 2 "" V 6230 7300 50  0001 C CNN
+F 2 "library_express_pro:R_1.2mm" V 6230 7300 50  0001 C CNN
 F 3 "~" H 6300 7300 50  0001 C CNN
 	1    6300 7300
@@
 F 0 "VoltageMonitor1" H 1075 3085 50  0000 C CNN
 F 1 "BD48K60" H 1075 3176 50  0000 C CNN
-F 2 "" H 1100 3200 50  0001 C CNN
+F 2 "library_express_pro:SSOP3" H 1100 3200 50  0001 C CNN
 F 3 "" H 1100 3200 50  0001 C CNN
 	1    1100 3300
@@
 F 0 "AI-1223-TWT-5V-5-R1" H 2408 3002 50  0000 L CNN
 F 1 "Buzzer" V 2499 3002 50  0000 L CNN
-F 2 "" V 2425 2950 50  0001 C CNN
+F 2 "library_express_pro:Buzzer_AI-1223-TWT-5V-5-R" V 2425 2950 50  0001 C CNN
 F 3 "~" V 2425 2950 50  0001 C CNN
 	1    2450 2850
@@
 F 0 "R_IR1" H 2520 6696 50  0001 L CNN
 F 1 "220" H 2380 6650 50  0001 R CNN
-F 2 "" V 2380 6650 50  0001 C CNN
+F 2 "library_express_pro:R_1.2mm" V 2380 6650 50  0001 C CNN
 F 3 "~" H 2450 6650 50  0001 C CNN
 	1    2450 6650
@@
 F 0 "2N7002K1" H 1806 7146 50  0000 L CNN
 F 1 "NMOS_DGS" H 1806 7055 50  0000 L CNN
-F 2 "Package_TO_SOT_SMD:SOT-23" H 1800 7200 50  0001 C CNN
+F 2 "library_express_pro:SOT23" H 1800 7200 50  0001 C CNN
 F 3 "~" H 1600 7100 50  0001 C CNN
 	1    1600 7100
@@
 F 0 "R4" V 1193 7300 50  0001 C CNN
 F 1 "10K" H 1284 7300 50  0000 C CNN
-F 2 "" V 1330 7300 50  0001 C CNN
+F 2 "library_express_pro:R_1.2mm" V 1330 7300 50  0001 C CNN
 F 3 "~" H 1400 7300 50  0001 C CNN
 	1    1400 7300
@@
 F 0 "R1" H 1820 5446 50  0000 L CNN
 F 1 "220" H 1680 5400 50  0000 R CNN
-F 2 "" V 1680 5400 50  0001 C CNN
+F 2 "library_express_pro:R_1.2mm" V 1680 5400 50  0001 C CNN
 F 3 "~" H 1750 5400 50  0001 C CNN
 	1    1750 5400
@@
 F 0 "R2" H 1820 5796 50  0000 L CNN
 F 1 "220" H 1680 5750 50  0000 R CNN
-F 2 "" V 1680 5750 50  0001 C CNN
+F 2 "library_express_pro:R_1.2mm" V 1680 5750 50  0001 C CNN
 F 3 "~" H 1750 5750 50  0001 C CNN
 	1    1750 5750
@@
 	10000 2900 9950 2900
 $Comp
-L Device:Q_PMOS_DSG SPD30P06P_G1
+L Device:Q_PMOS_DSG Si4101DY1
 U 1 1 5D1601C1
 P 1700 1000
-F 0 "SPD30P06P_G1" H 1906 1046 50  0000 L CNN
+F 0 "Si4101DY1" H 1906 1046 50  0000 L CNN
 F 1 "PMOS" H 1906 1000 50  0000 L CNN
-F 2 "Package_TO_SOT_SMD:TO-252-2" H 1900 1100 50  0001 C CNN
+F 2 "library_express_pro:SOT23" H 1900 1100 50  0001 C CNN
 F 3 "~" H 1700 1000 50  0001 C CNN
 	1    1700 1000

Commit message: some connectors footprints added
Parts:
- J3: footprint (none) -> library_express_pro:Accelerometer_standard
- MotorConnector1: footprint (none) -> library_express_pro:motor_connector
Changed lines of the file:
@@
 F 0 "MotorConnector1" H 8668 725 50  0000 C CNN
 F 1 "Conn_01x02" H 8668 816 50  0000 C CNN
-F 2 "" H 8750 1050 50  0001 C CNN
+F 2 "library_express_pro:motor_connector" H 8750 1050 50  0001 C CNN
 F 3 "~" H 8750 1050 50  0001 C CNN
 	1    8750 1050
@@
 F 0 "J3" H 9880 5342 50  0001 L CNN
 F 1 "Accelerometer_standard" H 9880 5296 50  0000 L CNN
-F 2 "" H 9800 5350 50  0001 C CNN
+F 2 "library_express_pro:Accelerometer_standard" H 9800 5350 50  0001 C CNN
 F 3 "~" H 9800 5350 50  0001 C CNN
 	1    9800 5350

Commit message: raspberry pin headers added for review
Parts:
- J1: footprint (none) -> library_express_pro:RaspberryPi_pins
Changed lines of the file:
@@
 F 0 "J1" V 9654 2013 50  0001 R CNN
 F 1 "Conn_02x20_Odd_Even" H 9745 2013 50  0000 R CNN
-F 2 "" H 9650 3100 50  0001 C CNN
+F 2 "library_express_pro:RaspberryPi_pins" H 9650 3100 50  0001 C CNN
 F 3 "~" H 9650 3100 50  0001 C CNN
 	1    9650 3100

Commit message: motor & power connector pending changes
Parts:
- J2: footprint (none) -> library_express_pro:accelerometer_small
- J4: footprint (none) -> library_express_pro:servo_connector
Changed lines of the file:
@@
 F 0 "J2" H 9880 4842 50  0001 L CNN
 F 1 "Accelerometer_small" H 9880 4796 50  0000 L CNN
-F 2 "" H 9800 4850 50  0001 C CNN
+F 2 "library_express_pro:accelerometer_small" H 9800 4850 50  0001 C CNN
 F 3 "~" H 9800 4850 50  0001 C CNN
 	1    9800 4850
@@
 F 0 "J4" H 9880 6092 50  0001 L CNN
 F 1 "Servo_motor" H 9880 6046 50  0000 L CNN
-F 2 "" H 9800 6050 50  0001 C CNN
+F 2 "library_express_pro:servo_connector" H 9800 6050 50  0001 C CNN
 F 3 "~" H 9800 6050 50  0001 C CNN
 	1    9800 6050

Commit message: working on PCB design
Parts:
- C1, C2, C3, C4, C5, C6, C7, C8, C9, L1: footprint (none) -> library_express_pro:RLC_EIA_3216
- LDO1: footprint Package_TO_SOT_SMD:TO-252-2 -> library_express_pro:TO252-2
- MotorConnector1: footprint library_express_pro:motor_connector -> library_express_pro:Connector_pads
- None1, YSL-R531R3D-D1, YSL-R531R3D-D2, YSL-R531R3D-D3, YSL-R531R3D-D4: footprint (none) -> library_express_pro:LED_YSL-R531R3D-D2
- Power1: footprint (none) -> library_express_pro:Connector_pads
- R1, R10, R11, R12, R13, R14, R1_buck1, R2, R2_buck1, R3, R4, R5, R7, R8, R9, R_IR1, Rmax1: footprint library_express_pro:R_1.2mm -> library_express_pro:RLC_EIA_3216
Changed lines of the file:
@@
 F 0 "C1" V 1252 3900 50  0001 C CNN
 F 1 "10uF" V 1160 3900 50  0000 C CNN
-F 2 "" H 1038 3750 50  0001 C CNN
+F 2 "library_express_pro:RLC_EIA_3216" H 1038 3750 50  0001 C CNN
 F 3 "~" H 1000 3900 50  0001 C CNN
 	1    1000 3900
@@
 F 0 "MotorConnector1" H 8668 725 50  0000 C CNN
 F 1 "Conn_01x02" H 8668 816 50  0000 C CNN
-F 2 "library_express_pro:motor_connector" H 8750 1050 50  0001 C CNN
+F 2 "library_express_pro:Connector_pads" H 8750 1050 50  0001 C CNN
 F 3 "~" H 8750 1050 50  0001 C CNN
 	1    8750 1050
@@
 F 0 "C3" H 1915 1596 50  0001 L CNN
 F 1 "100nF" H 1915 1550 50  0000 L CNN
-F 2 "" H 1838 1400 50  0001 C CNN
+F 2 "library_express_pro:RLC_EIA_3216" H 1838 1400 50  0001 C CNN
 F 3 "~" H 1800 1550 50  0001 C CNN
 	1    1800 1550
@@
 F 0 "C2" H 1082 1504 50  0001 R CNN
 F 1 "170uF" H 1082 1550 50  0000 R CNN
-F 2 "" H 1238 1400 50  0001 C CNN
+F 2 "library_express_pro:RLC_EIA_3216" H 1238 1400 50  0001 C CNN
 F 3 "~" H 1200 1550 50  0001 C CNN
 	1    1200 1550
@@
 F 0 "Rmax1" H 720 1196 50  0000 L CNN
 F 1 "280" H 720 1105 50  0000 L CNN
-F 2 "library_express_pro:R_1.2mm" V 580 1150 50  0001 C CNN
+F 2 "library_express_pro:RLC_EIA_3216" V 580 1150 50  0001 C CNN
 F 3 "~" H 650 1150 50  0001 C CNN
 	1    650  1150
@@
 F 0 "Power1" H 1180 642 50  0000 L CNN
 F 1 "Conn_01x02" H 1180 551 50  0000 L CNN
-F 2 "" H 1100 650 50  0001 C CNN
+F 2 "library_express_pro:Connector_pads" H 1100 650 50  0001 C CNN
 F 3 "~" H 1100 650 50  0001 C CNN
 	1    1100 650
@@
 F 0 "R3" V 4607 1400 50  0000 C CNN
 F 1 "100K" V 4516 1400 50  0000 C CNN
-F 2 "library_express_pro:R_1.2mm" V 4330 1400 50  0001 C CNN
+F 2 "library_express_pro:RLC_EIA_3216" V 4330 1400 50  0001 C CNN
 F 3 "~" H 4400 1400 50  0001 C CNN
 	1    4400 1400
@@
 F 0 "C6" V 5702 1300 50  0000 C CNN
 F 1 "0.1uF" V 5611 1300 50  0000 C CNN
-F 2 "" H 5488 1150 50  0001 C CNN
+F 2 "library_express_pro:RLC_EIA_3216" H 5488 1150 50  0001 C CNN
 F 3 "~" H 5450 1300 50  0001 C CNN
 	1    5450 1300
@@
 F 0 "L1" V 5519 1550 50  0000 C CNN
 F 1 "3.3uH" V 5610 1550 50  0000 C CNN
-F 2 "" H 5700 1550 50  0001 C CNN
+F 2 "library_express_pro:RLC_EIA_3216" H 5700 1550 50  0001 C CNN
 F 3 "~" H 5700 1550 50  0001 C CNN
 	1    5700 1550
@@
 F 0 "C9" H 6685 1654 50  0000 R CNN
 F 1 "44uF" H 6685 1745 50  0000 R CNN
-F 2 "" H 6838 1550 50  0001 C CNN
+F 2 "library_express_pro:RLC_EIA_3216" H 6838 1550 50  0001 C CNN
 F 3 "~" H 6800 1700 50  0001 C CNN
 	1    6800 1700
@@
 F 0 "R2_buck1" V 6307 2150 50  0001 C CNN
 F 1 "22.1K" V 6216 2150 50  0000 C CNN
-F 2 "library_express_pro:R_1.2mm" V 6030 2150 50  0001 C CNN
+F 2 "library_express_pro:RLC_EIA_3216" V 6030 2150 50  0001 C CNN
 F 3 "~" H 6100 2150 50  0001 C CNN
 	1    6100 2150
@@
 F 0 "C4" H 4185 2054 50  0000 R CNN
 F 1 "1uF" H 4185 2145 50  0000 R CNN
-F 2 "" H 4338 1950 50  0001 C CNN
+F 2 "library_express_pro:RLC_EIA_3216" H 4338 1950 50  0001 C CNN
 F 3 "~" H 4300 2100 50  0001 C CNN
 	1    4300 2100
@@
 F 0 "C5" H 5335 2454 50  0000 R CNN
 F 1 "1uF" H 5335 2545 50  0000 R CNN
-F 2 "" H 5488 2350 50  0001 C CNN
+F 2 "library_express_pro:RLC_EIA_3216" H 5488 2350 50  0001 C CNN
 F 3 "~" H 5450 2500 50  0001 C CNN
 	1    5450 2500
@@
 F 0 "R1_buck1" V 5893 1800 50  0001 C CNN
 F 1 "124k" V 5984 1800 50  0000 C CNN
-F 2 "library_express_pro:R_1.2mm" V 6030 1800 50  0001 C CNN
+F 2 "library_express_pro:RLC_EIA_3216" V 6030 1800 50  0001 C CNN
 F 3 "~" H 6100 1800 50  0001 C CNN
 	1    6100 1800
@@
 F 0 "YSL-R531R3D-D2" H 5893 5445 50  0000 C CNN
 F 1 "LED" H 5893 5536 50  0000 C CNN
-F 2 "" H 5900 5700 50  0001 C CNN
+F 2 "library_express_pro:LED_YSL-R531R3D-D2" H 5900 5700 50  0001 C CNN
 F 3 "~" H 5900 5700 50  0001 C CNN
 	1    5900 5700
@@
 F 0 "R5" V 1693 3350 50  0001 C CNN
 F 1 "10K" H 1784 3350 50  0000 C CNN
-F 2 "library_express_pro:R_1.2mm" V 1830 3350 50  0001 C CNN
+F 2 "library_express_pro:RLC_EIA_3216" V 1830 3350 50  0001 C CNN
 F 3 "~" H 1900 3350 50  0001 C CNN
 	1    1900 3350
@@
 F 0 "R8" H 4570 5896 50  0001 L CNN
 F 1 "220" H 4430 5850 50  0000 R CNN
-F 2 "library_express_pro:R_1.2mm" V 4430 5850 50  0001 C CNN
+F 2 "library_express_pro:RLC_EIA_3216" V 4430 5850 50  0001 C CNN
 F 3 "~" H 4500 5850 50  0001 C CNN
 	1    4500 5850
@@
 F 0 "R7" H 4570 5096 50  0001 L CNN
 F 1 "220" H 4430 5050 50  0000 R CNN
-F 2 "library_express_pro:R_1.2mm" V 4430 5050 50  0001 C CNN
+F 2 "library_express_pro:RLC_EIA_3216" V 4430 5050 50  0001 C CNN
 F 3 "~" H 4500 5050 50  0001 C CNN
 	1    4500 5050
@@
 F 0 "R9" H 4570 6646 50  0001 L CNN
 F 1 "220" H 4430 6600 50  0000 R CNN
-F 2 "library_express_pro:R_1.2mm" V 4430 6600 50  0001 C CNN
+F 2 "library_express_pro:RLC_EIA_3216" V 4430 6600 50  0001 C CNN
 F 3 "~" H 4500 6600 50  0001 C CNN
 	1    4500 6600
@@
 F 0 "R10" H 4570 7446 50  0001 L CNN
 F 1 "220" H 4430 7400 50  0000 R CNN
-F 2 "library_express_pro:R_1.2mm" V 4430 7400 50  0001 C CNN
+F 2 "library_express_pro:RLC_EIA_3216" V 4430 7400 50  0001 C CNN
 F 3 "~" H 4500 7400 50  0001 C CNN
 	1    4500 7400
@@
 F 0 "R11" H 6370 5746 50  0001 L CNN
 F 1 "82" H 6230 5700 50  0000 R CNN
-F 2 "library_express_pro:R_1.2mm" V 6230 5700 50  0001 C CNN
+F 2 "library_express_pro:RLC_EIA_3216" V 6230 5700 50  0001 C CNN
 F 3 "~" H 6300 5700 50  0001 C CNN
 	1    6300 5700
@@
 F 0 "YSL-R531R3D-D1" H 5893 5995 50  0000 C CNN
 F 1 "LED" H 5893 6086 50  0000 C CNN
-F 2 "" H 5900 6250 50  0001 C CNN
+F 2 "library_express_pro:LED_YSL-R531R3D-D2" H 5900 6250 50  0001 C CNN
 F 3 "~" H 5900 6250 50  0001 C CNN
 	1    5900 6250
@@
 F 0 "R12" H 6370 6296 50  0001 L CNN
 F 1 "82" H 6230 6250 50  0000 R CNN
-F 2 "library_express_pro:R_1.2mm" V 6230 6250 50  0001 C CNN
+F 2 "library_express_pro:RLC_EIA_3216" V 6230 6250 50  0001 C CNN
 F 3 "~" H 6300 6250 50  0001 C CNN
 	1    6300 6250
@@
 F 0 "YSL-R531R3D-D3" H 5893 6545 50  0000 C CNN
 F 1 "LED" H 5893 6636 50  0000 C CNN
-F 2 "" H 5900 6800 50  0001 C CNN
+F 2 "library_express_pro:LED_YSL-R531R3D-D2" H 5900 6800 50  0001 C CNN
 F 3 "~" H 5900 6800 50  0001 C CNN
 	1    5900 6800
@@
 F 0 "R13" H 6370 6846 50  0001 L CNN
 F 1 "82" H 6230 6800 50  0000 R CNN
-F 2 "library_express_pro:R_1.2mm" V 6230 6800 50  0001 C CNN
+F 2 "library_express_pro:RLC_EIA_3216" V 6230 6800 50  0001 C CNN
 F 3 "~" H 6300 6800 50  0001 C CNN
 	1    6300 6800
@@
 F 0 "YSL-R531R3D-D4" H 5893 7045 50  0000 C CNN
 F 1 "LED" H 5893 7136 50  0000 C CNN
-F 2 "" H 5900 7300 50  0001 C CNN
+F 2 "library_express_pro:LED_YSL-R531R3D-D2" H 5900 7300 50  0001 C CNN
 F 3 "~" H 5900 7300 50  0001 C CNN
 	1    5900 7300
@@
 F 0 "R14" H 6370 7346 50  0001 L CNN
 F 1 "82" H 6230 7300 50  0000 R CNN
-F 2 "library_express_pro:R_1.2mm" V 6230 7300 50  0001 C CNN
+F 2 "library_express_pro:RLC_EIA_3216" V 6230 7300 50  0001 C CNN
 F 3 "~" H 6300 7300 50  0001 C CNN
 	1    6300 7300
@@
 F 0 "R_IR1" H 2520 6696 50  0001 L CNN
 F 1 "220" H 2380 6650 50  0001 R CNN
-F 2 "library_express_pro:R_1.2mm" V 2380 6650 50  0001 C CNN
+F 2 "library_express_pro:RLC_EIA_3216" V 2380 6650 50  0001 C CNN
 F 3 "~" H 2450 6650 50  0001 C CNN
 	1    2450 6650
@@
 F 0 "None1" H 2143 6395 50  0001 C CNN
 F 1 "IR_LED" H 2143 6486 50  0000 C CNN
-F 2 "" H 2150 6650 50  0001 C CNN
+F 2 "library_express_pro:LED_YSL-R531R3D-D2" H 2150 6650 50  0001 C CNN
 F 3 "~" H 2150 6650 50  0001 C CNN
 	1    2150 6650
@@
 F 0 "R4" V 1193 7300 50  0001 C CNN
 F 1 "10K" H 1284 7300 50  0000 C CNN
-F 2 "library_express_pro:R_1.2mm" V 1330 7300 50  0001 C CNN
+F 2 "library_express_pro:RLC_EIA_3216" V 1330 7300 50  0001 C CNN
 F 3 "~" H 1400 7300 50  0001 C CNN
 	1    1400 7300
@@
 F 0 "C7" H 6235 1754 50  0000 R CNN
 F 1 "44uF" H 6235 1845 50  0000 R CNN
-F 2 "" H 6388 1650 50  0001 C CNN
+F 2 "library_express_pro:RLC_EIA_3216" H 6388 1650 50  0001 C CNN
 F 3 "~" H 6350 1800 50  0001 C CNN
 	1    6350 1800
@@
 F 0 "LDO1" H 1225 5825 50  0000 C CNN
 F 1 "AZ2085" H 1225 5734 50  0000 C CNN
-F 2 "Package_TO_SOT_SMD:TO-252-2" H 1200 5100 50  0001 C CNN
+F 2 "library_express_pro:TO252-2" H 1200 5100 50  0001 C CNN
 F 3 "" H 1200 5100 50  0001 C CNN
 	1    1200 5400
@@
 F 0 "R1" H 1820 5446 50  0000 L CNN
 F 1 "220" H 1680 5400 50  0000 R CNN
-F 2 "library_express_pro:R_1.2mm" V 1680 5400 50  0001 C CNN
+F 2 "library_express_pro:RLC_EIA_3216" V 1680 5400 50  0001 C CNN
 F 3 "~" H 1750 5400 50  0001 C CNN
 	1    1750 5400
@@
 F 0 "R2" H 1820 5796 50  0000 L CNN
 F 1 "220" H 1680 5750 50  0000 R CNN
-F 2 "library_express_pro:R_1.2mm" V 1680 5750 50  0001 C CNN
+F 2 "library_express_pro:RLC_EIA_3216" V 1680 5750 50  0001 C CNN
 F 3 "~" H 1750 5750 50  0001 C CNN
 	1    1750 5750
@@
 F 0 "C8" V 2352 5400 50  0001 C CNN
 F 1 "10uF" V 2260 5400 50  0000 C CNN
-F 2 "" H 2138 5250 50  0001 C CNN
+F 2 "library_express_pro:RLC_EIA_3216" H 2138 5250 50  0001 C CNN
 F 3 "~" H 2100 5400 50  0001 C CNN
 	1    2100 5400

Commit message: PCB Board first layout
Parts:
- SW1, SW2, SW3, SW4: footprint (none) -> library_express_pro:button_6x6mm
Changed lines of the file:
@@
 F 0 "SW2" H 4100 5925 50  0001 C CNN
 F 1 "SW_DPST" H 4100 5834 50  0001 C CNN
-F 2 "" H 4100 5600 50  0001 C CNN
+F 2 "library_express_pro:button_6x6mm" H 4100 5600 50  0001 C CNN
 F 3 "~" H 4100 5600 50  0001 C CNN
 	1    4100 5600
@@
 F 0 "SW1" H 4100 5125 50  0001 C CNN
 F 1 "SW_DPST" H 4100 5034 50  0001 C CNN
-F 2 "" H 4100 4800 50  0001 C CNN
+F 2 "library_express_pro:button_6x6mm" H 4100 4800 50  0001 C CNN
 F 3 "~" H 4100 4800 50  0001 C CNN
 	1    4100 4800
@@
 F 0 "SW3" H 4100 6675 50  0001 C CNN
 F 1 "SW_DPST" H 4100 6584 50  0001 C CNN
-F 2 "" H 4100 6350 50  0001 C CNN
+F 2 "library_express_pro:button_6x6mm" H 4100 6350 50  0001 C CNN
 F 3 "~" H 4100 6350 50  0001 C CNN
 	1    4100 6350
@@
 F 0 "SW4" H 4100 7475 50  0001 C CNN
 F 1 "SW_DPST" H 4100 7384 50  0001 C CNN
-F 2 "" H 4100 7150 50  0001 C CNN
+F 2 "library_express_pro:button_6x6mm" H 4100 7150 50  0001 C CNN
 F 3 "~" H 4100 7150 50  0001 C CNN
 	1    4100 7150

Commit message: PCB board in the works
Parts:
- J1: footprint library_express_pro:RaspberryPi_pins -> library_express_pro:RasPi_header_pro
Changed lines of the file:
@@
 F 0 "J1" V 9654 2013 50  0001 R CNN
 F 1 "Conn_02x20_Odd_Even" H 9745 2013 50  0000 R CNN
-F 2 "library_express_pro:RaspberryPi_pins" H 9650 3100 50  0001 C CNN
+F 2 "library_express_pro:RasPi_header_pro" H 9650 3100 50  0001 C CNN
 F 3 "~" H 9650 3100 50  0001 C CNN
 	1    9650 3100

Commit message: Night Session
Parts:
- added H1, H2, H3, H4: MountingHole, MountingHole:MountingHole_2.7mm_M2.5, symbol Mechanical:MountingHole
- Si4101DY1: footprint library_express_pro:SOT23 -> library_express_pro:SO-8
Changed lines of the file:
@@
 F 0 "Si4101DY1" H 1906 1046 50  0000 L CNN
 F 1 "PMOS" H 1906 1000 50  0000 L CNN
-F 2 "library_express_pro:SOT23" H 1900 1100 50  0001 C CNN
+F 2 "library_express_pro:SO-8" H 1900 1100 50  0001 C CNN
 F 3 "~" H 1700 1000 50  0001 C CNN
 	1    1700 1000
 	1    0    0    -1
 $EndComp
+$Comp
+L Mechanical:MountingHole H1
+U 1 1 5D325F07
+P 6350 700
+F 0 "H1" H 6450 746 50  0000 L CNN
+F 1 "MountingHole" H 6450 655 50  0000 L CNN
+F 2 "MountingHole:MountingHole_2.7mm_M2.5" H 6350 700 50  0001 C CNN
+F 3 "~" H 6350 700 50  0001 C CNN
+	1    6350 700
+	1    0    0    -1
+$EndComp
+$Comp
+L Mechanical:MountingHole H3
+U 1 1 5D326A35
+P 7100 700
+F 0 "H3" H 7200 746 50  0000 L CNN
+F 1 "MountingHole" H 7200 655 50  0000 L CNN
+F 2 "MountingHole:MountingHole_2.7mm_M2.5" H 7100 700 50  0001 C CNN
+F 3 "~" H 7100 700 50  0001 C CNN
+	1    7100 700
+	1    0    0    -1
+$EndComp
+$Comp
+L Mechanical:MountingHole H2
+U 1 1 5D33042E
+P 6350 900
+F 0 "H2" H 6450 946 50  0000 L CNN
+F 1 "MountingHole" H 6450 855 50  0000 L CNN
+F 2 "MountingHole:MountingHole_2.7mm_M2.5" H 6350 900 50  0001 C CNN
+F 3 "~" H 6350 900 50  0001 C CNN
+	1    6350 900
+	1    0    0    -1
+$EndComp
+$Comp
+L Mechanical:MountingHole H4
+U 1 1 5D339C5C
+P 7100 900
+F 0 "H4" H 7200 946 50  0000 L CNN
+F 1 "MountingHole" H 7200 855 50  0000 L CNN
+F 2 "MountingHole:MountingHole_2.7mm_M2.5" H 7100 900 50  0001 C CNN
+F 3 "~" H 7100 900 50  0001 C CNN
+	1    7100 900
+	1    0    0    -1
+$EndComp
