File: first_design/_autosave-first_design.sch (KiCad schematic (older format))
At the start: 56 parts, among them J1 Conn_02x20_Odd_Even, J2 Accelerometer_small, J3 Accelerometer_standard, J4 Servo_motor

Commit message: board
Parts:
- SQJA37EP1: footprint (none) -> library_express_pro:SO-8L
Changed lines of the file:
@@
 F 0 "SQJA37EP1" H 1906 1046 50  0000 L CNN
 F 1 "PMOS" H 1906 1000 50  0000 L CNN
-F 2 "" H 1900 1100 50  0001 C CNN
+F 2 "library_express_pro:SO-8L" H 1900 1100 50  0001 C CNN
 F 3 "~" H 1700 1000 50  0001 C CNN
 	1    1700 1000
