File: first_design/_autosave-first_design.sch (KiCad schematic (older format))
At the start: 43 parts, among them IC1 BD48K60, IC2 AZ2085D-ADJTRG1, IC3 AP65450, IC5 VNH7070BAS, J1 Conn_02x20_Odd_Even, J2 Conn_01x02, J3 Accelerometer_standard, J4 Servo_motor, J5 Battery, Q1 2N7002K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

Commit message: Ready for PCB Prototyping
Parts:
- renumbered IR_LED1 to IRD1
Connections:
- net GPIO20: now also Btn1.2
- net GPIO21: now also Btn2.2; no longer Btn1.2
- net GPIO26: no longer Btn2.2
Changed lines of the file:
@@
 $EndComp
 $Comp
-L Device:LED IR_LED1
+L Device:LED IRD1
 U 1 1 5D78C6B1
 P 2150 6650
-F 0 "IR_LED1" H 2143 6395 50  0000 C CNN
+F 0 "IRD1" H 2143 6395 50  0000 C CNN
 F 1 "IR_LED" H 2143 6486 50  0001 C CNN
 F 2 "library_express_pro:LED_YSL-R531R3D-D2" H 2150 6650 50  0001 C CNN
@@
 $EndComp
 Text GLabel 5550 5950 2    50   Input ~ 0
-GPIO21
+GPIO20
 Text GLabel 10150 4650 2    50   Input ~ 0
 GPIO12
@@
 $EndComp
 Text GLabel 5550 6300 2    50   Input ~ 0
-GPIO26
+GPIO21
 Wire Wire Line
 	5350 5950 5550 5950
