File: first_design/first_design.kicad_pcb (KiCad board)
At the start: 2 copper layers, 65 x 56.5 mm, 45 parts, among them IC1 BD48K60, IC2 AZ2085, IC3 AP65450, IC4 RN, IC5 VNH7070BAS, J1 Conn_02x20_Odd_Even, J3 Accelerometer_standard, J4 Servo_motor, Q1 Q_PMOS_DGS

Commit message: still finalizing
Parts:
- removed the Q1 at (30.0, -10.0)
- added Q2: DMG2301L, library_express_pro:SOT23, F.Cu at (30.0, -8.00)
- Btn1: renamed from Button1; value led1 -> PTS636
- Btn2: value led2 -> PTS636
- Btn3: value led3 -> PTS636
- Btn4: value led4 -> PTS636
- LED1: renamed from YSL-R531R3D-D2; value LED1 -> 599-0210-007F
- LED2: renamed from YSL-R531R3D-D1; value LED2 -> 599-0210-007F
- LED3: renamed from YSL-R531R3D-D3; value LED3 -> 599-0210-007F
- LED4: renamed from YSL-R531R3D-D4; value LED4 -> 599-0210-007F
- LS1: renamed from AI1027TWT5V2R1; value Buzzer -> AI1027TWT5V2R
- Q1: renamed from 2N7002K1; value NMOS_DGS -> 2N7002K
- Q3: renamed from SQJA37EP1; value PMOS -> SQJA37EP1
- RN1: renamed from IC4; value RN -> YC324_JK_07220RL
- renumbered None1 to IR_LED1, MotorConnector1 to J2, R1_buck1 to R5, R2_buck1 to R6, R_IR1 to R7, R_IR2 to R8
Connections:
- net +3.3V renamed +3V3
Routing:
- net Net-(JP2-Pad1): track 4.41 -> 7.26 mm
- net +5V: track 75.9 -> 77.2 mm
- net Net-(IC1-Pad1): track 15.4 -> 16.1 mm

Commit message: Ready for PCB Prototyping
Parts:
- removed Btn3, Btn4: PTS636, library_express_pro:PTS636
- removed C6: 0.1uF, library_express_pro:RLC_EIA_3216
- removed LED3, LED4: 599-0210-007F, library_express_pro:RLC_EIA_3216
- removed RN1: YC324_JK_07220RL, library_express_pro:Resistor_array_YC324
- added C1: 10uF 25V, Pi HAT Footprints:CAPC320X160X180L50M, F.Cu at (32.0, -27.0)
- added C3: 1uF 25V, Pi HAT Footprints:CAPC320X160X180L50M, F.Cu at (27.5, -19.5)
- added R10: 220, library_express_pro:RLC_EIA_3216, F.Cu at (60.5, -24.0)
- added R9: 220, library_express_pro:RLC_EIA_3216, F.Cu at (52.0, -24.0)
- C4, C5: value 1uF -> 1uF 25V; footprint library_express_pro:RLC_EIA_3216 -> Pi HAT Footprints:CAPC320X160X180L50M
- C9: value 44uF -> 22uF 25V; footprint library_express_pro:Capacitor_E61 -> Pi HAT Footprints:CAPC320X250X180L50L
- IC2: value AZ2085 -> AZ2085D-ADJTRG1; footprint library_express_pro:TO252-2 -> Pi HAT Footprints:DPAK3P457_1010X238L155X81T525X470M
- IC3: footprint library_express_pro:SO-8 -> Pi HAT Footprints:SOIC9P127_490X600X150L72X40T305X241L
- IC5: footprint library_express_pro:SO-16N -> Pi HAT Footprints:SOIC16P127_990X600X175L83X41M
- J5: renamed from Power1; value Conn_01x02 -> Battery
- JP2, JP3, JP4: moved to B.Cu
- L1: footprint library_express_pro:Inductor_PA4340 -> Pi HAT Footprints:INDC800X800X450L240M
- Q2: value DMG2301L -> DMG2301L-7
- R4, R6: value 22.1K -> 22.1k
- moved R4 22.2 mm to (42.3, -43.4), turned to 180 degrees
- moved JP4 16.1 mm to (32.0, -3.50)
- moved Q2 15.6 mm to (41.5, -18.5)
- moved C9 14.6 mm to (35.5, -27.0), turned to 90 degrees
- moved Q1 14.4 mm to (42.2, -38.9), turned to 90 degrees
- moved R1 14.1 mm to (13.5, -14.0)
- moved R5 14.1 mm to (16.5, -23.5), turned to 90 degrees
- moved JP1 14.0 mm to (37.5, -4.00)
- moved LED1 13.3 mm to (52.0, -30.5)
- moved J4 12.0 mm to (26.0, -10.5)
- moved C4 12.0 mm to (23.0, -32.5), turned to 270 degrees
- moved LED2 11.9 mm to (60.5, -30.5)
- moved IC1 11.7 mm to (33.5, -3.50), turned to 0 degrees
- moved IC2 10.9 mm to (13.5, -4.50), turned to 90 degrees
- moved C2 10.5 mm to (23.0, -27.0)
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- renumbered IR_LED1 to IRD1
Connections:
- net VCC renamed Net-(J5-Pad1)
- Btn1 pad 2: GPIO21 -> GPIO20
- Btn2 pad 2: GPIO26 -> GPIO21
- C2 pad 2: Vbat -> +BATT
- C4 pad 1: GND -> Net-(C4-Pad1)
- IC1 pad 2: Vbat -> +BATT
- IC2 pad 3: Vbat -> +BATT
- IC3 pad 1: Vbat -> +BATT
- IC3 pad 4: Net-(C4-Pad2) -> Net-(C3-Pad2)
- IC3 pad 6: Net-(C6-Pad2) -> Net-(C4-Pad1)
- IC3 pad 7: Net-(C6-Pad1) -> Net-(C4-Pad2)
- IC3 pad 8: Vbat -> +BATT
- L1 pad 2: Net-(C6-Pad2) -> Net-(C4-Pad1)
- LED1 pad 2: GPIO5 -> GPIO16
- LED2 pad 2: GPIO6 -> GPIO26
- Q1 pad 1: Net-(IR_LED1-Pad1) -> Net-(IRD1-Pad1)
- Q3 pad 2: Vbat -> +BATT
- R7 pad 1: Net-(IR_LED1-Pad2) -> Net-(IRD1-Pad2)
Routing:
- net GPIO25: track 48.8 -> 0.00 mm
- net GPIO13: track 42.1 -> 0.00 mm
- net Net-(LED4-Pad1): track 36.1 -> 0.00 mm
- net +BATT: track 0.00 -> 30.6 mm, vias 0 -> 10
- net GPIO20: track 38.7 -> 9.75 mm
- net Net-(LED3-Pad1): track 28.5 -> 0.00 mm
- net GPIO16: track 50.2 -> 24.1 mm
- net Vbat: track 27.8 -> 4.85 mm, vias 14 -> 6
- net +3V3: track 110.9 -> 88.9 mm
- net GPIO6: track 20.3 -> 0.00 mm
- net Net-(LED2-Pad1): track 19.9 -> 3.45 mm
- net GPIO8: track 36.8 -> 21.2 mm, vias 2 -> 0
- net Net-(IC1-Pad1): track 16.1 -> 27.2 mm, vias 0 -> 1
- net +5V: track 77.2 -> 67.6 mm, vias 7 -> 5
- net Net-(LED1-Pad1): track 12.8 -> 3.43 mm
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- added copper zone on B.Cu, net +BATT
- added copper zone on F.Cu, net +BATT
- added copper zone on F.Cu, net Net-(C4-Pad1)
- removed copper zone on F.Cu, net Net-(C6-Pad2)
- removed copper zone on F.Cu, net Net-(J4-Pad2)
- removed copper zone on B.Cu, net Vbat
- removed copper zone on F.Cu, net Vservo
Other:
- rule trace_min: 0.15 -> 0.2
