File: first_design/RaceOn-PiHAT.sch (KiCad schematic (older format))
At the start: 62 parts, among them J1 Conn_02x20_Odd_Even, J2 Conn_01x02, J3 Accelerometer_standard, J4 Servo_motor, J5 Battery, Q3 SQJA37EP1

Commit message: Renamed project to RaceOn-PiHAT
Other:
- note added: "Servo Power Supply"
Changed lines of the file:
@@
 $EndComp
 Text Notes 7300 4400 0    157  ~ 0
-Motor Controller
+Servo Power Supply
 $Comp
 L RaceOn-PiHAT:NCP5901B IC?
@@
 Wire Wire Line
 	9100 4850 9100 5650
+Text Notes 6350 750  0    157  ~ 0
+Motor Controller
 $EndSCHEMATC
