File: RaceOn-PiHAT.sch (KiCad schematic (older format))
At the start: 77 parts, among them IC1 MIC29302WU, IC10 SN74LVC2G07, IC2 NCP5901B, IC3 NCP5901B, IC4 BD48K60G, IC5 LMR14030, IC6 MPU-9250, IC7 SN74LVC2G07, IC8 SN74LVC2G07, IC9 SN74LVC2G07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

Commit message: Finished board
Parts:
- IC5: footprint Race On:SOIC9P127_490X600X170L83X41T287X202M -> Race On:SOIC9P127_490X600X170L83X41T287X202
Other:
- moved on the sheet: C12, C13, C15, C7, C8, D2, IC5, L1, R10, R8, R9

Commit message: Rev 1.3 final
Parts:
- added FID1: Fiducial, Race On:FID1M3, symbol Mechanical:Fiducial
Changed lines of the file:
@@
+	1    0    0    -1
+$EndComp
+$Comp
+L Mechanical:Fiducial FID1
+U 1 1 5E0E375F
+P 4200 6700
+F 0 "FID1" H 4285 6746 50  0000 L CNN
+F 1 "Fiducial" H 4285 6655 50  0000 L CNN
+F 2 "Race On:FID1M3" H 4200 6700 50  0001 C CNN
+F 3 "~" H 4200 6700 50  0001 C CNN
+	1    4200 6700
 	1    0    0    -1
 $EndComp
