File: _autosave-RaceOn-PiHAT.sch (KiCad schematic (older format))
At the start: 75 parts, among them IC1 MIC29302WU, IC10 SN74LVC2G07, IC2 NCP5901B, IC3 NCP5901B, IC4 BD48K60G, IC5 LMR14030, IC6 MPU-9250, IC7 SN74LVC2G07, IC8 SN74LVC2G07, IC9 SN74LVC2G07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

Commit message: Latest version
Parts:
- M1: MPN NOT IN OPL -> A2543WV-3P
Changed lines of the file:
@@
 F 2 "Race On:HDRV3W64P254_3X1_762X254H854" H 3400 1160 50  0001 C CNN
 F 3 "" H 3400 1160 50  0001 C CNN
-F 4 "NOT IN OPL" H 3400 1150 20  0000 C CNN "MPN"
+F 4 "A2543WV-3P" H 3400 1150 20  0000 C CNN "MPN"
 	1    3400 1350
 	1    0    0    -1
